File: test_arena_v1r2/test_arena_v1r2.kicad_sch (KiCad schematic)
At the start: 48 parts, among them J1 Conn_01x05_Socket, J2 Conn_01x05_Socket, J3 Barrel_Jack, U1 Teensy4.1, U2 SN74LV1T34DBV, U3 74LVC2G17, U4 74LVC2G17, U5 74LVC2G17, U6 74LVC2G17

Commit message: Added final design for modified test arena.
Parts:
- added TP11, TP12: TestPoint, TestPoint:TestPoint_THTPad_D2.0mm_Drill1.0mm, symbol Connector:TestPoint
Connections:
- net D30: now reaches U1.22 (30_CRX3)
- net D30: now also TP11.1
- net D31: now reaches U1.23 (31_CTX3)
- net D31: now also TP12.1
- no-connect marks 37 -> 35
Other:
- moved on the sheet: C6, C7, C8, C9, J1, J2, R10, R11, R12, R7, R8, R9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

Commit message: Added production files for v1r2 test arena.
Parts:
- C9: LCSC Part # C1525 -> C84455
- J3, U1: now not fitted; now left out of the parts list
- JP1: FT Rotation Offset (none) -> 90; LCSC Part # (none) -> C492401
- R1, R10, R11, R12, R2, R3, R4, R5, R6, R7, R8, R9: LCSC Part # (none) -> C25105
- U3, U4, U5, U6: LCSC Part # (none) -> C7836
Other:
- note removed: "Add Teensy GPIO test points!"

Commit message: Fixed wrong part issue on v1r2  test arena.
Parts:
- U3, U4, U5, U6: LCSC Part # C7836 -> C10429
Changed lines of the file:
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@@
 			)
 		)
-		(property "LCSC Part #" "C7836"
+		(property "LCSC Part #" "C10429"
 			(at 293.37 142.24 0)
 			(effects
@@
 			)
 		)
-		(property "LCSC Part #" "C7836"
+		(property "LCSC Part #" "C10429"
 			(at 196.85 62.23 0)
 			(effects
@@
 			)
 		)
-		(property "LCSC Part #" "C7836"
+		(property "LCSC Part #" "C10429"
 			(at 41.91 66.04 0)
 			(effects
@@
 			)
 		)
-		(property "LCSC Part #" "C7836"
+		(property "LCSC Part #" "C10429"
 			(at 41.91 81.28 0)
 			(effects
@@
 			)
 		)
-		(property "LCSC Part #" "C7836"
+		(property "LCSC Part #" "C10429"
 			(at 196.85 142.24 0)
 			(effects
@@
 			)
 		)
-		(property "LCSC Part #" "C7836"
+		(property "LCSC Part #" "C10429"
 			(at 196.85 90.17 0)
 			(effects
@@
 			)
 		)
-		(property "LCSC Part #" "C7836"
+		(property "LCSC Part #" "C10429"
 			(at 196.85 34.29 0)
 			(effects
@@
 			)
 		)
-		(property "LCSC Part #" "C7836"
+		(property "LCSC Part #" "C10429"
 			(at 245.11 142.24 0)
 			(effects
@@
 			)
 		)
-		(property "LCSC Part #" "C7836"
+		(property "LCSC Part #" "C10429"
 			(at 35.56 114.3 0)
 			(effects
@@
 			)
 		)
-		(property "LCSC Part #" "C7836"
+		(property "LCSC Part #" "C10429"
 			(at 196.85 76.2 0)
 			(effects
@@
 			)
 		)
-		(property "LCSC Part #" "C7836"
+		(property "LCSC Part #" "C10429"
 			(at 196.85 104.14 0)
 			(effects
@@
 			)
 		)
-		(property "LCSC Part #" "C7836"
+		(property "LCSC Part #" "C10429"
 			(at 196.85 48.26 0)
 			(effects
